Commit message: Nav2 Stack configuration

File: src/myrobot_description/urdf/robot/my_robot_gazebo.xacro (robot description, xacro)
@@ -141,3 +141,31 @@
     </sensor>
   </gazebo>
+  <!-- Camera -->
+  <gazebo reference="camera_link">
+    <sensor name="camera" type="camera">
+      <always_on>true</always_on>
+      <update_rate>30</update_rate>
+      <visualize>true</visualize>
+      <topic>camera/image_raw</topic>
+      <camera>
+        <horizontal_fov>1.047</horizontal_fov>
+        <image>
+          <width>700</width>
+          <height>600</height>
+        </image>
+        <clip>
+          <near>0.1</near>
+          <far>100</far>
+        </clip>
+        <distortion>
+          <k1>0</k1>
+          <k2>0</k2>
+          <k3>0</k3>
+          <p1>0</p1>
+          <p2>0</p2>
+          <center>0.5 0.5</center>
+        </distortion>
+      </camera>
+    </sensor>
+  </gazebo>
 </robot>

File: src/myrobot_description/urdf/robot/my_robot_homemade.xacro (robot description, xacro)
@@ -4,5 +4,5 @@
   <xacro:property name="base_length" value="0.20" />
   <xacro:property name="base_width" value="0.30" />
-  <xacro:property name="base_height" value="0.10" />
+  <xacro:property name="base_height" value="0.30" />
   <xacro:property name="base_mass" value="1.0" />
   <xacro:property name="wheel_mass" value="0.3" />
@@ -10,5 +10,5 @@
   <xacro:property name="wheel_length" value="0.02" />
   <xacro:property name="caster_wheel_mass" value="0.1" />
-  <xacro:property name="caster_wheel_radius" value="0.015" />
+  <xacro:property name="caster_wheel_radius" value="${wheel_radius / 2.0}" />
   <!-- BASE FOOTPRINT LINK -->
   <link name="base_footprint" />
@@ -136,4 +136,21 @@
     </xacro:inertial_cylinder>
   </link>
+  <!-- CAMERA LINK -->
+  <link name="camera_link">
+    <visual>
+      <geometry>
+        <box size="0.05 0.05 0.05"/>
+      </geometry>
+      <material name="red"/>
+    </visual>
+    <collision>
+      <geometry>
+        <box size="0.05 0.05 0.05"/>
+      </geometry>
+    </collision>
+    <xacro:inertial_box mass="0.1" x="0.05" y="0.05" z="0.05">
+      <origin xyz="0 0 0" rpy="0 0 0"/>
+    </xacro:inertial_box>
+  </link>
   <!-- JOINTS -->
   <joint name="base_joint" type="fixed">
@@ -175,3 +192,9 @@
     <origin xyz="0 0 ${base_height + 0.057 / 2.0}" rpy="0 0 0"/>
   </joint>
+  <joint name="camera_joint" type="fixed">
+    <parent link="base_link"/>
+    <child link="camera_link"/>
+    <!-- Positioned near the front edge of the top plate, facing forward -->
+    <origin xyz="${base_length/2} 0 ${base_height - 0.1}" rpy="0 0.5235987756 0"/>
+  </joint>
 </robot>

File: src/myrobot_description/urdf/robot/robot_ros2_control.xacro (robot description, xacro)
@@ -27,6 +27,6 @@
         <joint name="right_wheel_joint">
             <command_interface name="velocity">
-                <param name="min">-1</param>
-                <param name="max">1</param>
+                <param name="min">-20</param>
+                <param name="max">20</param>
             </command_interface>
             <state_interface name="position" />
@@ -35,6 +35,6 @@
         <joint name="left_wheel_joint">
             <command_interface name="velocity">
-                <param name="min">-1</param>
-                <param name="max">1</param>
+                <param name="min">-20</param>
+                <param name="max">20</param>
             </command_interface>
             <state_interface name="position" />
