Commit message: Nav2 Simulation Cleanup

File: src/myrobot_description/urdf/robot/my_robot.urdf.xacro (robot description, xacro)
@@ -5,5 +5,4 @@
     <xacro:include filename="common_properties.xacro" />
     <xacro:include filename="my_robot_homemade.xacro" />
-    <!--xacro:include filename="mobile_base_printed.xacro" /-->
     <xacro:include filename="robot_ros2_control.xacro" />
     <xacro:include filename="my_robot_gazebo.xacro" />

File: src/myrobot_description/urdf/robot/my_robot_gazebo.xacro (robot description, xacro)
@@ -39,14 +39,4 @@
   <!-- ROS 2 Control -->
   <gazebo>
-    <!-- ROS 2 Humble -->
-    <xacro:if value="$(arg is_ignition)">
-      <plugin filename="ign_ros2_control-system" name="ign_ros2_control::IgnitionROS2ControlPlugin">
-        <parameters>$(find myrobot_controller)/config/myrobot_controllers.yaml</parameters>
-      </plugin>
-      <plugin filename="ignition-gazebo-imu-system" name="ignition::gazebo::systems::Imu">
-      </plugin>
-    </xacro:if>
-    <!-- ROS 2 Iron or above -->
-    <xacro:unless value="$(arg is_ignition)">
       <plugin filename="gz_ros2_control-system" name="gz_ros2_control::GazeboSimROS2ControlPlugin">
         <parameters>$(find myrobot_controller)/config/myrobot_controllers.yaml</parameters>
@@ -54,5 +44,7 @@
       <plugin filename="gz-sim-imu-system" name="gz::sim::systems::Imu">
       </plugin>
-    </xacro:unless>
+      <plugin filename="gz-sim-sensors-system" name="gz::sim::systems::Sensors">
+        <render_engine>ogre2</render_engine>
+      </plugin>
   </gazebo>
   <!-- IMU -->

File: src/myrobot_description/urdf/robot/my_robot_homemade.xacro (robot description, xacro)
@@ -196,5 +196,5 @@
     <child link="camera_link"/>
     <!-- Positioned near the front edge of the top plate, facing forward -->
-    <origin xyz="${base_length/2} 0 ${base_height - 0.1}" rpy="0 0.5235987756 0"/>
+    <origin xyz="${base_length/2} 0 ${base_height - 0.1}" rpy="0 0 0"/>
   </joint>
 </robot>

File: src/myrobot_description/urdf/robot/robot_ros2_control.xacro (robot description, xacro)
@@ -2,25 +2,9 @@
 <robot xmlns:xacro="http://www.ros.org/wiki/xacro" name="my_robot">
     <ros2_control name="RobotSystem" type="system">
-        <!-- ros2_control Real Robot -->
-        <xacro:unless value="$(arg is_sim)">
-            <hardware>
-                <plugin>myrobot_firmware/MyRobotInterface</plugin>
-                <param name="port">/dev/ttyUSB0</param>
-            </hardware>
-        </xacro:unless>
         <!-- ros2_control Gazebo -->
         <xacro:if value="$(arg is_sim)">
-            <!-- ROS 2 Humble -->
-            <xacro:if value="$(arg is_ignition)">
-                <hardware>
-                    <plugin>ign_ros2_control/IgnitionSystem</plugin>
-                </hardware>
-            </xacro:if>
-            <!-- ROS 2 Iron or above -->
-            <xacro:unless value="$(arg is_ignition)">
-                <hardware>
-                    <plugin>gz_ros2_control/GazeboSimSystem</plugin>
-                </hardware>
-            </xacro:unless>
+            <hardware>
+                <plugin>gz_ros2_control/GazeboSimSystem</plugin>
+            </hardware>
         </xacro:if>
         <!-- ros2_control Common Interfaces -->
